File: RP2350B-RM2.kicad_pcb (KiCad board)
At the start: 2 copper layers, 52 x 89.5 mm, 57 parts, among them J1 10103594-0001LF, J2 Conn_01x29, J3 Conn_01x28, J4 SM03B-SRSS-TB(LF)(SN), SW1 434133025816, SW2 434133025816, U1 RP2350B, U2 NCP1117ST33T3G, U3 W25Q128JVSIQ, U4 APS6404L-3SQR-SN, U5 RM2, X1 12MHz

Commit message: Remove the J4 debug connector; route SWD/SWCLK straight to J3
SWD and SWCLK are on J3 (pins 22/23, next to RUN), so the JST debug
connector is redundant.

Schematic: J4, its wiring, its GND symbol and the "JST Debug Connector"
heading are removed. SWD/SWCLK keep their labels at U1 and J3.

Board (edited on top of the refilled board): J4, its GND stubs and two
vias, and the "DEBUG" silkscreen are removed. Pi ran SWD and SWCLK
through J4's pads; they now continue along the same 45-degree lines
into their existing horizontal runs to J3. Zones refilled.

Pipeline: update_pcb_from_sch.py now deletes footprints whose symbol is
gone, and layout_rm2.py has the matching J4 section. Re-running both from
Pi's original board reproduces this board exactly (same footprints,
tracks, vias and zones). The layout script's docstring is brought up to
date.

DRC: 0 unconnected items, 0 parity issues, 45 RPI_COMPILED library
notes. ERC unchanged (4 pre-existing items). The J4 BOM line is removed.

Co-Authored-By: Claude Opus 5.5 <noreply@anthropic.com>
Claude-Session: https://claude.ai/code/session_01TVxWe2rd4mhh6Q8D57QZer
Parts:
- removed J4: SM03B-SRSS-TB(LF)(SN), RPI_COMPILED:jst_sm03b-srss-tb-lf--sn-
Routing:
- net GND: track 54.6 -> 48.5 mm, vias 39 -> 37
- net /SWCLK: track 38.9 -> 37.7 mm
Other:
- board text removed: "DEBUG"
