File: RP2350B-RM2.kicad_sch (KiCad schematic)
At the start: 59 parts, among them J1 10103594-0001LF, J2 Conn_01x29, J3 Conn_01x28, SW1 434133025816, SW2 434133025816, U1 RP2350B, U2 NCP1117ST33T3G, U3 W25Q128JVSIQ, U4 APS6404L-3SQR-SN, U5 RM2, X1 12MHz

Commit message: Add a 5 V VSYS input on J3 pin 2, with USB VBUS through a Schottky
J3 pin 2 (was a second 3V3 pin) is now VSYS, the input of the 3.3 V
regulator, so the board can run from 5 V on the header without USB.
USB VBUS reaches VSYS through D2 (B5819W, SOD-123), so header power
can't back-feed a connected computer, as on a Pico.

- Schematic: D2 between VBUS and VSYS, a VSYS power symbol and a
  PWR_FLAG; J3 pin 2's power symbol is VSYS.
- PCB: D2 sits between J1, C1 and U2. Pi's VBUS pour is split into a
  USB side (J1 to D2's anode) and VSYS. A 0.6 mm VSYS track runs from
  D2's cathode through U2's input pad, under U2 and up to J3 pin 2, so
  the 3V3 pour around J3 pin 1 stays joined to U2's output. Silkscreen
  label VSYS. layout_rm2.py reproduces the board from Pi's original.
- README power section, BOM line for D2 (LCSC C8598), renders.

DRC: 0 unconnected items, 0 schematic-parity issues. ERC: the same
pre-existing items as before.

Co-Authored-By: Claude Opus 5.5 <noreply@anthropic.com>
Claude-Session: https://claude.ai/code/session_01TVxWe2rd4mhh6Q8D57QZer
Parts:
- added D2: B5819W, Diode_SMD:D_SOD-123, symbol Device:D_Schottky
Connections:
- net +3V3: no longer J3.2 (Pin_2)
- net VBUS: now also D2.2 (A); no longer C1.1, U2.3 (IN)
- new net VSYS: C1.1, D2.1 (K), J3.2 (Pin_2), U2.3 (IN)
Other:
- note added: "VSYS is also J3 pin 2: run the board from 5 V there. D2 keeps that 5 V off the USB port; USB still powers the board through D2."
